File: pcb/teensy-jst_01.4 v10.brd (EAGLE design)
At the start: 66 x 105.4 mm, 91 parts, among them U1 TPS54360DDARDDA8_3P1X2P4_TEX

Commit message: teensy PCB with correct capacitor footprints
Parts:
- C10, C11: device rcl:C0805 -> Capacitor:CAPC2012X110
- C14, C15, C16, C17, C22, C8, C9: device rcl:C0402 -> Capacitor:CAPC1005X60
- C18, C19, C20, C21, C23, C24, C25, C26, C27: device rcl:C0402K -> Capacitor:CAPC1005X60
- C28, C3, C4, C5, C6, C7: device rcl:C0603 -> Capacitor:CAPC1608X85
- moved R26 0.25 mm to (-24.6, 78.4)
- moved C25 0.25 mm to (19.6, 48.3)
- moved C7 0.25 mm to (-21.6, 82.1)
- moved R21 0.25 mm to (19.3, 49.5)
- moved C8 0.18 mm to (-22.3, 84.6)
Other:
- board text added: "Cameron Chaney (c) 9/2025"
- board text removed: "Cameron Chaney (c) 8/2025"
