File: pcb/teensy-jst_01.4_v6.sch (EAGLE design)
At the start: 91 parts, among them U1 TPS54360DDARDDA8_3P1X2P4_TEX

Commit message: teensy PCB with correct capacitor footprints
Parts:
- C10, C11: device rcl:C-EUC0805 -> Capacitor:C_CHIP-0805(2012-METRIC)
- C14, C15, C16, C17, C22, C8, C9: device rcl:C-EUC0402 -> Capacitor:C_CHIP-0402(1005-METRIC)
- C18, C19, C20, C21, C23, C24, C25, C26, C27: device rcl:C-EUC0402K -> Capacitor:C_CHIP-0402(1005-METRIC)
- C28, C3, C4, C5, C6, C7: device rcl:C-EUC0603 -> Capacitor:C_CHIP-0603(1608-METRIC)
